Commit message: Add python config file and simple demo with pybullet

File: urdf/plane_with_restitution.urdf (robot description, URDF)
Before this commit: robot plane, 1 links, 0 joints
Links:
- link planeLink: geometry collision box size=30 30 10; visual mesh filename=package://teststand/meshes/plane.obj scale=1 1 1

File: xacro/teststand.urdf.xacro (robot description, xacro)
@@ -5,7 +5,7 @@
   xmlns:sensor="http://playerstage.sourceforge.net/gazebo/xmlschema/#sensor"
   xmlns:xacro="http://playerstage.sourceforge.net/gazebo/xmlschema/#interface">
-  <xacro:property name="base_w" value=".2" />
+  <xacro:property name="base_w" value=".1" />
   <xacro:property name="base_l" value=".2" />
-  <xacro:property name="base_h" value=".2" />
+  <xacro:property name="base_h" value=".1" />
   <xacro:property name="base_m" value="0.485" />
   <xacro:include filename="$(find robot_properties_teststand)/xacro_include/leg.xacro" />
@@ -13,10 +13,10 @@
    <joint name="joint_z" type="prismatic">
     <parent link="root"/>
-    <child link="base"/>
+    <child link="base_link"/>
     <limit effort="1000" lower="-10" upper="10" velocity="1000"/>
     <axis xyz="0 0 1"/>
     <origin rpy="0 0 0" xyz="0 0 0"/>
   </joint>
-  <link name="base">
+  <link name="base_link">
     <inertial>
         <origin rpy="0 0 0" xyz="0 0 ${base_h/2.}"/>
