Commit message: Fix xacro_include/leg.xacro - replace quadruped references with teststand

File: xacro_include/leg.xacro (robot description, xacro)
@@ -23,5 +23,5 @@
         <geometry>
             <!-- <cylinder length="${upper_leg_length}" radius="${upper_leg_radius}"/> -->
-            <mesh filename="package://robot_properties_quadruped/meshes/cylinder.obj" scale="${upper_leg_radius} ${upper_leg_radius} ${upper_leg_length}"/>
+            <mesh filename="package://robot_properties_teststand/meshes/cylinder.obj" scale="${upper_leg_radius} ${upper_leg_radius} ${upper_leg_length}"/>
         </geometry>
         <material name="grey">
@@ -61,5 +61,5 @@
         <geometry>
             <!-- <cylinder length="${upper_leg_length}" radius="${upper_leg_radius}"/> -->
-            <mesh filename="package://robot_properties_quadruped/meshes/cylinder.obj" scale="${upper_leg_radius} ${upper_leg_radius} ${upper_leg_length}"/>
+            <mesh filename="package://robot_properties_teststand/meshes/cylinder.obj" scale="${upper_leg_radius} ${upper_leg_radius} ${upper_leg_length}"/>
         </geometry>
         <material name="grey">
@@ -96,5 +96,5 @@
         <geometry>
             <!-- <sphere radius="${upper_leg_radius}"/> -->
-            <mesh filename="package://robot_properties_quadruped/meshes/sphere.obj" scale="${upper_leg_radius} ${upper_leg_radius} ${upper_leg_radius}"/>
+            <mesh filename="package://robot_properties_teststand/meshes/sphere.obj" scale="${upper_leg_radius} ${upper_leg_radius} ${upper_leg_radius}"/>
         </geometry>
         <material name="red">

Commit message: Make TeststandConfig.buildRobotWrapper include visual shapes. Update leg parts to use stls also used on solo

File: xacro_include/leg.xacro (robot description, xacro)
@@ -5,115 +5,160 @@
   xmlns:sensor="http://playerstage.sourceforge.net/gazebo/xmlschema/#sensor"
   xmlns:xacro="http://playerstage.sourceforge.net/gazebo/xmlschema/#interface">
-    <xacro:property name="upper_leg_length" value="0.16" />
-    <xacro:property name="upper_leg_radius" value="0.025" />
-    <xacro:property name="upper_leg_mass" value="0.162" />
-    <xacro:property name="lower_leg_mass" value="0.021" />
-    <xacro:macro name="leg" params="prefix rx ry">
+  <xacro:property name="color_name" value="grey" />
+  <xacro:property name="color" value="0.8 0.8 0.8" />
+  <xacro:property name="opacity" value="1.0" />
+  <xacro:property name="mesh_ext" value="stl" />
+  <!-- See TODO: add the wiki link here -->
+  <!-- These are absoulte distance value, the sign are decided below -->
+  <xacro:property name="base_2_HFE_x" value="${190.00 * 0.001}" />
+  <xacro:property name="base_2_HFE_y" value="${104.60 * 0.001}" />
+  <xacro:property name="HFE_2_KFE_y" value="${37.45 * 0.001}" />
+  <xacro:property name="HFE_2_KFE_z" value="${160.00 * 0.001}" />
+  <xacro:property name="KFE_2_FOOT_y" value="${8.0 * 0.001}" />
+  <xacro:property name="KFE_2_FOOT_z" value="${160.00 * 0.001}" />
+  <xacro:macro name="leg" params="prefix ry rx">
+    <!-- Joint between the base and the ${prefix} upper leg -->
     <joint name="${prefix}HFE" type="revolute">
-        <parent link="base_link"/>
-        <child link="${prefix}upperleg"/>
-        <limit effort="1000" lower="-10" upper="10" velocity="1000"/>
-        <axis xyz="0 1 0"/>
-        <origin rpy="0 0 0" xyz="${rx} ${ry} 0"/>
-        <dynamics damping="0.0" friction="0.0"/>
+      <parent link="base_link"/>
+      <child link="${prefix}upperleg"/>
+      <limit effort="1000" lower="-10" upper="10" velocity="1000"/>
+      <!-- joints rotates around the y-axis -->
+      <axis xyz="0 1 0"/>
+      <!-- placement of the joint -->
+      <origin xyz="${rx} ${ry} 0" rpy="0 0 0" />
+      <!-- pybullet simulation parameters -->
+      <dynamics damping="0.0" friction="0.0"/>
     </joint>
     <link name="${prefix}upperleg">
-        <visual>
-        <origin rpy="0 0 0" xyz="0 0 ${-.5*upper_leg_length}"/>
+      <!-- UPPER LEG LINK INERTIAL -->
+      <!-- Left upper leg inertia -->
+      <inertial>
+        <origin xyz="0.00001377 0.01935853 -0.07870700" rpy="0 0 0" />
+        <mass value="0.14853845"/>
+        <inertia ixx="0.00041107" ixy="0.0"         ixz="0.0"
+                                   iyy="0.00041193" iyz="0.00004671"
+                                                    izz="0.00003024"/>
+      </inertial>
+      <!-- UPPER LEG LINK VISUAL -->
+      <visual>
+        <origin xyz="0 0 0" rpy="0 0 0" />
         <geometry>
-            <!-- <cylinder length="${upper_leg_length}" radius="${upper_leg_radius}"/> -->
-            <mesh filename="package://robot_properties_teststand/meshes/cylinder.obj" scale="${upper_leg_radius} ${upper_leg_radius} ${upper_leg_length}"/>
+            <mesh filename="package://robot_properties_teststand/meshes/${mesh_ext}/with_foot/solo_upper_leg_left_side.${mesh_ext}"/>
         </geometry>
-        <material name="grey">
-            <color rgba=".4 .4 .4 .1"/>
+        <material name="${color_name}">
+            <color rgba="${color} ${opacity}"/>
         </material>
-        </visual>
-        <collision>
-        <origin rpy="0 0 0" xyz="0 0 ${-.5*upper_leg_length}"/>
+      </visual>
+      <!-- UPPER LEG LINK COLLISION -->
+      <collision>
+        <origin xyz="0 0 0" rpy="0 0 0" />
         <geometry>
-            <cylinder length="${upper_leg_length}" radius="${upper_leg_radius}"/>
+            <mesh filename="package://robot_properties_teststand/meshes/${mesh_ext}/with_foot/solo_upper_leg_left_side.${mesh_ext}"/>
         </geometry>
-        </collision>
-        <inertial>
-        <origin rpy="0 0 0" xyz="0 0 -0.0793"/>
-        <mass value="${upper_leg_mass}"/>
-        <inertia ixy="0.0" ixz="0.0" iyz="0.0"
-            ixx="0.000469609"
-            iyy="0.000469609"
-            izz="1e-6"/>
-        </inertial>
-    </link>
+        <material name="${color_name}">
+            <color rgba="${color} ${opacity}"/>
+        </material>
+      </collision>
+      <!-- Bullet specific paramters -->
+      <contact>
+        <lateral_friction value="1.0"/>
+        <restitution value="0.5"/>
+      </contact>
+    </link> <!-- END UPPER LEG LINK -->
+    <!-- KFE: Joint between the upper leg and the lower leg -->
     <joint name="${prefix}KFE" type="revolute">
-        <parent link="${prefix}upperleg"/>
-        <child link="${prefix}shank"/>
-        <limit effort="1000" velocity="10000"/>
-        <axis xyz="0 1 0"/>
-        <origin rpy="0 0 0" xyz="0 0 ${-upper_leg_length}"/>
-        <dynamics damping="0.0" friction="0.0"/>
+      <parent link="${prefix}upperleg"/>
+      <child link="${prefix}shank"/>
+      <limit effort="1000" lower="-10" upper="10" velocity="1000"/>
+      <!-- joints rotates around the y-axis -->
+      <axis xyz="0 1 0"/>
+      <!-- placement of the joint -->
+      <origin xyz="0 ${HFE_2_KFE_y} ${-HFE_2_KFE_z}" rpy="0 0 0" />
+      <!-- pybullet simulation parameters -->
+      <dynamics damping="0.0" friction="0.0"/>
     </joint>
     <link name="${prefix}shank">
-        <contact>
-            <lateral_friction value="1.0"/>
-            <restitution value="0.5"/>
-        </contact>
-        <visual>
-        <origin rpy="0 0 0" xyz="0 0 ${-.5*upper_leg_length}"/>
+      <!-- LOWER LEG LINK INERTIAL -->
+      <!-- Left lower leg inertia -->
+      <inertial>
+        <origin xyz="0.0 0.00787644 -0.08928215" rpy="0 0 0" />
+        <mass value="0.03070001"/>
+        <inertia ixx="0.00012024" ixy="0.0"         ixz="0.0"
+                                   iyy="0.00012029" iyz="0.00000305"
+                                                    izz="0.00000216"/>
+      </inertial>
+      <!-- LOWER LEG LINK VISUAL -->
+      <visual>
+        <origin xyz="0 0 0" rpy="0 0 0" />
         <geometry>
-            <!-- <cylinder length="${upper_leg_length}" radius="${upper_leg_radius}"/> -->
-            <mesh filename="package://robot_properties_teststand/meshes/cylinder.obj" scale="${upper_leg_radius} ${upper_leg_radius} ${upper_leg_length}"/>
+          <mesh filename="package://robot_properties_teststand/meshes/${mesh_ext}/with_foot/solo_lower_leg_left_side.${mesh_ext}"/>
         </geometry>
-        <material name="grey">
-            <color rgba=".4 .4 .4 .1"/>
+        <material name="${color_name}">
+            <color rgba="${color} ${opacity}"/>
         </material>
-        </visual>
-        <collision>
-        <origin rpy="0 0 0" xyz="0 0 ${-.5*upper_leg_length}"/>
+      </visual>
+      <!-- LOWER LEG LINK COLLISION -->
+      <collision>
+        <origin xyz="0 0 0" rpy="0 0 0" />
         <geometry>
-            <cylinder length="${upper_leg_length}" radius="${upper_leg_radius}"/>
+          <mesh filename="package://robot_properties_teststand/meshes/${mesh_ext}/with_foot/solo_lower_leg_left_side.${mesh_ext}"/>
         </geometry>
-        </collision>
-        <inertial>
-        <origin rpy="0 0 0" xyz="0 0 -0.0756"/>
-        <mass value="${lower_leg_mass}"/>
-        <inertia ixy="0.0" ixz="0.0" iyz="0.0"
-            ixx="0.000087575"
-            iyy="0.000087575"
-            izz="1e-6"/>
-    </inertial>
-    </link>
+        <material name="${color_name}">
+            <color rgba="${color} ${opacity}"/>
+        </material>
+      </collision>
+      <!-- Bullet specific paramters -->
+      <contact>
+        <lateral_friction value="1.0"/>
+        <restitution value="0.5"/>
+      </contact>
+    </link> <!-- END LOWER LEG LINK -->
+    <!-- KFE: Joint between the upper leg and the lower leg -->
     <joint name="${prefix}END" type="fixed">
-        <parent link="${prefix}shank"/>
-        <child link="${prefix}contact"/>
-        <origin rpy="0 0 0" xyz="0 0 ${-upper_leg_length}"/>
+      <parent link="${prefix}shank"/>
+      <child link="${prefix}contact"/>
+      <!-- Joint placement -->
+      <origin xyz="0 ${KFE_2_FOOT_y} ${-KFE_2_FOOT_z}" rpy="0 0 0" />
+      <!-- Limits (usefull?) -->
+      <limit effort="1000" lower="-10" upper="10" velocity="1000"/>
+      <!-- pybullet simulation parameters -->
+      <dynamics damping="0.0" friction="0.0"/>
     </joint>
     <link name="${prefix}contact">
-        <contact>
-            <lateral_friction value="1.0"/>
-            <restitution value="0.5"/>
-        </contact>
-        <visual>
-        <origin rpy="0 0 0" xyz="0 0 0"/>
+      <!-- FOOT INERTIAL -->
+      <!-- This link is symmetrical left or right -->
+      <inertial>
+        <origin xyz="0 0 0.00035767" rpy="0 0 0" />
+        <mass value="0.00693606"/>
+        <inertia ixx="0.00000057" ixy="0.0"         ixz="0.0"
+                                   iyy="0.00000084" iyz="0.0"
+                                                    izz="0.00000053"/>
+     </inertial>
+      <!-- FOOT VISUAL -->
+      <visual>
+        <origin xyz="0 0 0" rpy="0 0 0" />
         <geometry>
-            <!-- <sphere radius="${upper_leg_radius}"/> -->
-            <mesh filename="package://robot_properties_teststand/meshes/sphere.obj" scale="${upper_leg_radius} ${upper_leg_radius} ${upper_leg_radius}"/>
+          <mesh filename="package://robot_properties_teststand/meshes/${mesh_ext}/with_foot/solo_foot.${mesh_ext}"/>
         </geometry>
-        <material name="red">
-            <color rgba="1. 0. 0. 1."/>
+        <material name="${color_name}">
+            <color rgba="${color} ${opacity}"/>
         </material>
-        </visual>
-        <collision>
-        <origin rpy="0 0 0" xyz="0 0 0"/>
+      </visual>
+      <!-- FOOT COLLISION -->
+      <collision>
+        <origin xyz="0 0 0" rpy="0 0 0" />
         <geometry>
-            <sphere radius="${upper_leg_radius}"/>
+            <mesh filename="package://robot_properties_teststand/meshes/${mesh_ext}/with_foot/solo_foot.${mesh_ext}"/>
         </geometry>
-        </collision>
-        <inertial>
-        <mass value="0.01"/>
-        <inertia ixy="0.0" ixz="0.0" iyz="0.0"
-            ixx="0."
-            iyy="0."
-            izz="0."/>
-    </inertial>
-    </link>
-    </xacro:macro>
+        <material name="${color_name}">
+            <color rgba="${color} ${opacity}"/>
+        </material>
+      </collision>
+      <!-- Bullet specific paramters -->
+      <contact>
+        <lateral_friction value="1.0"/>
+        <restitution value="0.5"/>
+      </contact>
+    </link> <!-- END LOWER LEG LINK -->
+  </xacro:macro>
 </robot>
