Commit message: made repo pip installable

File: src/robot_properties_teststand/resources/pre_generated_urdf/teststand.urdf (robot description, URDF)
Before this commit: robot teststand, 4 links, 3 joints
Links:
- removed link base
- added link base_link, mass 0.485; collision box size=0.2 0.1 0.1; visual mesh filename=package://meshes/cube.obj scale=0.2 0.1 0.1
- added link root
- link contact: geometry collision mesh filename=package://meshes/stl/with_foot/solo_foot.stl; visual mesh filename=package://meshes/stl/with_foot/solo_foot.stl
- link shank: geometry collision mesh filename=package://meshes/stl/with_foot/solo_lower_leg_left_side.stl; visual mesh filename=package://meshes/stl/with_foot/solo_lower_leg_left_side.stl
- link upperleg: geometry collision mesh filename=package://meshes/stl/with_foot/solo_upper_leg_left_side.stl; visual mesh filename=package://meshes/stl/with_foot/solo_upper_leg_left_side.stl
Joints:
- added joint joint_z: type prismatic, parent root, child base_link, origin xyz=0 0 0 rpy=0 0 0, axis 0 0 1, limit lower=-10 upper=10 effort=1000 velocity=1000

File: src/robot_properties_teststand/resources/xacro/leg.xacro (robot description, xacro)
@@ -44,5 +44,5 @@
         <origin xyz="0 0 0" rpy="0 0 0" />
         <geometry>
-            <mesh filename="package://robot_properties_teststand/meshes/${mesh_ext}/with_foot/solo_upper_leg_left_side.${mesh_ext}"/>
+            <mesh filename="package://meshes/${mesh_ext}/with_foot/solo_upper_leg_left_side.${mesh_ext}"/>
         </geometry>
         <material name="${color_name}">
@@ -54,5 +54,5 @@
         <origin xyz="0 0 0" rpy="0 0 0" />
         <geometry>
-            <mesh filename="package://robot_properties_teststand/meshes/${mesh_ext}/with_foot/solo_upper_leg_left_side.${mesh_ext}"/>
+            <mesh filename="package://meshes/${mesh_ext}/with_foot/solo_upper_leg_left_side.${mesh_ext}"/>
         </geometry>
         <material name="${color_name}">
@@ -92,5 +92,5 @@
         <origin xyz="0 0 0" rpy="0 0 0" />
         <geometry>
-          <mesh filename="package://robot_properties_teststand/meshes/${mesh_ext}/with_foot/solo_lower_leg_left_side.${mesh_ext}"/>
+          <mesh filename="package://meshes/${mesh_ext}/with_foot/solo_lower_leg_left_side.${mesh_ext}"/>
         </geometry>
         <material name="${color_name}">
@@ -102,5 +102,5 @@
         <origin xyz="0 0 0" rpy="0 0 0" />
         <geometry>
-          <mesh filename="package://robot_properties_teststand/meshes/${mesh_ext}/with_foot/solo_lower_leg_left_side.${mesh_ext}"/>
+          <mesh filename="package://meshes/${mesh_ext}/with_foot/solo_lower_leg_left_side.${mesh_ext}"/>
         </geometry>
         <material name="${color_name}">
@@ -139,5 +139,5 @@
         <origin xyz="0 0 0" rpy="0 0 0" />
         <geometry>
-          <mesh filename="package://robot_properties_teststand/meshes/${mesh_ext}/with_foot/solo_foot.${mesh_ext}"/>
+          <mesh filename="package://meshes/${mesh_ext}/with_foot/solo_foot.${mesh_ext}"/>
         </geometry>
         <material name="${color_name}">
@@ -149,5 +149,5 @@
         <origin xyz="0 0 0" rpy="0 0 0" />
         <geometry>
-            <mesh filename="package://robot_properties_teststand/meshes/${mesh_ext}/with_foot/solo_foot.${mesh_ext}"/>
+            <mesh filename="package://meshes/${mesh_ext}/with_foot/solo_foot.${mesh_ext}"/>
         </geometry>
         <material name="${color_name}">

File: src/robot_properties_teststand/resources/xacro/teststand.urdf.xacro (robot description, xacro)
@@ -31,5 +31,5 @@
         <origin rpy="0 0 0" xyz="0 0 ${base_h/2.}"/>
         <geometry>
-          <mesh filename="package://robot_properties_teststand/meshes/cube.obj" scale="${base_l} ${base_w} ${base_h}"/>
+          <mesh filename="package://meshes/cube.obj" scale="${base_l} ${base_w} ${base_h}"/>
         </geometry>
         <material name="white">
