Commit message: included package name in the mesh path in xacro files; renamed yaml_path to dgm_yaml_path; removed xacro encodings for python2

File: src/robot_properties_teststand/robot_properties_teststand/xacro/leg.xacro (robot description, xacro)
@@ -44,5 +44,5 @@
         <origin xyz="0 0 0" rpy="0 0 0" />
         <geometry>
-            <mesh filename="package://meshes/${mesh_ext}/with_foot/solo_upper_leg_left_side.${mesh_ext}"/>
+            <mesh filename="package://robot_properties_teststand/meshes/${mesh_ext}/with_foot/solo_upper_leg_left_side.${mesh_ext}"/>
         </geometry>
         <material name="${color_name}">
@@ -54,5 +54,5 @@
         <origin xyz="0 0 0" rpy="0 0 0" />
         <geometry>
-            <mesh filename="package://meshes/${mesh_ext}/with_foot/solo_upper_leg_left_side.${mesh_ext}"/>
+            <mesh filename="package://robot_properties_teststand/meshes/${mesh_ext}/with_foot/solo_upper_leg_left_side.${mesh_ext}"/>
         </geometry>
         <material name="${color_name}">
@@ -92,5 +92,5 @@
         <origin xyz="0 0 0" rpy="0 0 0" />
         <geometry>
-          <mesh filename="package://meshes/${mesh_ext}/with_foot/solo_lower_leg_left_side.${mesh_ext}"/>
+          <mesh filename="package://robot_properties_teststand/meshes/${mesh_ext}/with_foot/solo_lower_leg_left_side.${mesh_ext}"/>
         </geometry>
         <material name="${color_name}">
@@ -102,5 +102,5 @@
         <origin xyz="0 0 0" rpy="0 0 0" />
         <geometry>
-          <mesh filename="package://meshes/${mesh_ext}/with_foot/solo_lower_leg_left_side.${mesh_ext}"/>
+          <mesh filename="package://robot_properties_teststand/meshes/${mesh_ext}/with_foot/solo_lower_leg_left_side.${mesh_ext}"/>
         </geometry>
         <material name="${color_name}">
@@ -139,5 +139,5 @@
         <origin xyz="0 0 0" rpy="0 0 0" />
         <geometry>
-          <mesh filename="package://meshes/${mesh_ext}/with_foot/solo_foot.${mesh_ext}"/>
+          <mesh filename="package://robot_properties_teststand/meshes/${mesh_ext}/with_foot/solo_foot.${mesh_ext}"/>
         </geometry>
         <material name="${color_name}">
@@ -149,5 +149,5 @@
         <origin xyz="0 0 0" rpy="0 0 0" />
         <geometry>
-            <mesh filename="package://meshes/${mesh_ext}/with_foot/solo_foot.${mesh_ext}"/>
+            <mesh filename="package://robot_properties_teststand/meshes/${mesh_ext}/with_foot/solo_foot.${mesh_ext}"/>
         </geometry>
         <material name="${color_name}">

File: src/robot_properties_teststand/robot_properties_teststand/xacro/teststand.urdf.xacro (robot description, xacro)
@@ -31,5 +31,5 @@
         <origin rpy="0 0 0" xyz="0 0 ${base_h/2.}"/>
         <geometry>
-          <mesh filename="package://meshes/cube.obj" scale="${base_l} ${base_w} ${base_h}"/>
+          <mesh filename="package://robot_properties_teststand/meshes/cube.obj" scale="${base_l} ${base_w} ${base_h}"/>
         </geometry>
         <material name="white">
